File: nano_cnc_shield.kicad_pcb (KiCad board)
At the start: 2 copper layers, 19 parts, among them J1 POWER_12V, J2 LASER, J3 STEPPER_X, J4 STEPPER_Y, Q1 IRFZ44N, SW1 POWER_SWITCH, U1 L7805

Commit message: finished layout
Parts:
- added MH1: MountingHole_3.2mm_M3_DIN965, MountingHole:MountingHole_3.2mm_M3_DIN965, F.Cu at (40.0, 60.0)
- added MH2: MountingHole_3.2mm_M3_DIN965, MountingHole:MountingHole_3.2mm_M3_DIN965, F.Cu at (124.0, 60.0)
- moved JP1 115.1 mm to (52.7, 60.0)
- moved A2 113.5 mm to (44.4, 77.0)
- moved J3 113.4 mm to (49.5, 82.0)
- moved A3 112.0 mm to (67.3, 77.0), turned to 90 degrees
- moved SW1 80.0 mm to (120.5, 40.0), turned to 180 degrees
- moved D1 78.5 mm to (110.0, 40.0), turned to 180 degrees
- moved JP2 77.1 mm to (61.6, 60.0)
- moved R3 74.3 mm to (91.1, 40.0)
- moved JP3 69.8 mm to (75.6, 60.0), turned to 180 degrees
- moved JP4 67.5 mm to (84.4, 60.0)
- moved R1 64.1 mm to (91.1, 45.0)
- moved R2 63.4 mm to (91.1, 50.0)
- moved J4 62.1 mm to (72.4, 82.0), turned to 90 degrees
- moved J1 61.6 mm to (120.5, 48.0), turned to -90 degrees
- moved Q1 55.3 mm to (110.0, 65.0)
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Other:
- board outline added: 90 x 53 mm
- board text added: "+"
- board text added: "+12V"
- board text added: "-"
- board text added: "10k"
- board text added: "1A"
- board text added: "1B"
- board text added: "1k"
- board text added: "2A"
- board text added: "2B"
- board text added: "47"
- board text added: "A4988"
- board text added: "Arduino Nano"
- board text added: "EN_X"
- board text added: "EN_Y"
- board text added: "GND"
- board text added: "IRFZ44N"
- board text added: "LM7805"
- board text added: "OFF"
- board text added: "ON"
- board text added: "SLEEP_X"
- board text added: "SLEEP_Y"
- board text added: "X"
- board text added: "Y"
- board text added: "https://github.com/KacperBizon/nano_cnc_shield"

Commit message: add general routing
Parts:
- added C2: 100uF, Capacitor_THT:CP_Radial_D8.0mm_P3.50mm, F.Cu at (60.5, 70.7)
- added C3: 100uF, Capacitor_THT:CP_Radial_D8.0mm_P3.50mm, F.Cu at (83.4, 70.7)
- moved Q1 19.0 mm to (92.0, 59.0), turned to -90 degrees
- moved C1 15.5 mm to (105.0, 50.5)
- moved R1 3.21 mm to (87.9, 45.0)
- moved R2 3.21 mm to (87.9, 50.0)
- moved R3 3.21 mm to (87.9, 40.0)
- turned SW1 to 0 degrees
Routing:
- net GND: track 0.00 -> 135.5 mm, vias 0 -> 4
- net +12V: track 0.00 -> 102.4 mm
- net +5V: track 0.00 -> 75.2 mm, vias 0 -> 1
- net /X_STEP: track 0.00 -> 37.8 mm
- net /X_DIR: track 0.00 -> 35.7 mm
- net /LASER_SIGNAL: track 0.00 -> 35.1 mm
- net /Y_DIR: track 0.00 -> 31.5 mm
- net /Y_STEP: track 0.00 -> 29.4 mm
- net Net-(J1-V+): track 0.00 -> 24.5 mm
- net Net-(J2-Pin_2): track 0.00 -> 16.2 mm
- net Net-(D1-A): track 0.00 -> 9.38 mm
- net Net-(A3-~{RESET}): track 0.00 -> 6.84 mm
- net Net-(A2-~{RESET}): track 0.00 -> 6.84 mm
- net Net-(A3-2B): track 0.00 -> 5.00 mm
- net Net-(A3-2A): track 0.00 -> 5.00 mm
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Other:
- board text added: "100uF"

Commit message: final layout
Routing:
- net GND: track 135.5 -> 205.2 mm, vias 4 -> 7
- net Net-(J2-Pin_2): track 16.2 -> 71.5 mm, vias 0 -> 1
- net Net-(J2-Pin_1): track 0.00 -> 38.9 mm
- net Net-(Q1-G): track 0.00 -> 16.5 mm
- net /LASER_SIGNAL: track 35.1 -> 48.9 mm
- net (no net): vias 0 -> 1
- added copper zone on B.Cu, net GND
- added copper zone on F.Cu, net GND
Other:
- board text added: "1000uF"
- board text added: "LASER"

Commit message: flip LM7805, move heatsink pads
Parts:
- added MH3: MountingHole_2.7mm_M2.5_DIN965_Pad, MountingHole:MountingHole_2.7mm_M2.5_DIN965_Pad, F.Cu at (92.3, 80.8)
- added MH4: MountingHole_2.7mm_M2.5_DIN965_Pad, MountingHole:MountingHole_2.7mm_M2.5_DIN965_Pad, F.Cu at (117.7, 80.8)
- moved U1 5.08 mm to (107.5, 78.0), turned to 180 degrees
Routing:
- net +12V: track 102.4 -> 108.5 mm
- net Net-(J2-Pin_2): track 71.5 -> 67.0 mm
- net GND: track 205.2 -> 208.6 mm
Other:
- outline, holes or cut-outs redrawn
